Commit message: feat:Add Slider Control

File: mycobot_description/urdf/mycobot.xacro (robot description, xacro)
@@ -134,5 +134,5 @@
         </geometry>
         <origin xyz="0 0 0 " rpy="0 0 0" />
-        <material name="white" />
+        <material name="green" />
       </visual>
       <collision>

Commit message: fix:m5atom2.3->2.4

File: mycobot_description/urdf/mycobot.xacro (robot description, xacro)
@@ -134,5 +134,5 @@
         </geometry>
         <origin xyz="0 0 0 " rpy="0 0 0" />
-        <material name="green" />
+        <material name="white" />
       </visual>
       <collision>
@@ -155,5 +155,5 @@
         </geometry>
         <origin xyz="0 0.0025 0" rpy="${M_PI/2} 0 0" />
-        <material name="white" />
+        <material name="green" />
       </visual>
       <collision>
